File: kicad/commandpod/commandpod.sch (KiCad schematic (older format))
At the start: 1 part

Commit message: Annotated schematics
Parts:
- gave numbers to parts that had none: 1
Changed lines of the file:
@@
 $EndDescr
 $Comp
-L PHOTON PH?
+L PHOTON PH1
 U 1 1 56BF15F2
 P 5500 4000
-F 0 "PH?" H 5350 3350 60  0001 C CNN
+F 0 "PH1" H 5350 3350 60  0001 C CNN
 F 1 "PHOTON" V 5500 4000 60  0000 C CNN
 F 2 "~" H 5460 4160 60  0000 C CNN
@@
 NoConn ~ 6050 3950
 $Comp
-L +3.3V #PWR?
+L +3.3V #PWR01
 U 1 1 56D62628
 P 6250 3300
-F 0 "#PWR?" H 6250 3260 30  0001 C CNN
+F 0 "#PWR01" H 6250 3260 30  0001 C CNN
 F 1 "+3.3V" H 6250 3410 30  0000 C CNN
 F 2 "" H 6250 3300 60  0000 C CNN
@@
 $EndComp
 $Comp
-L +5V #PWR?
+L +5V #PWR02
 U 1 1 56D6267B
 P 4750 3300
-F 0 "#PWR?" H 4750 3390 20  0001 C CNN
+F 0 "#PWR02" H 4750 3390 20  0001 C CNN
 F 1 "+5V" H 4750 3390 30  0000 C CNN
 F 2 "" H 4750 3300 60  0000 C CNN
@@
 $EndComp
 $Comp
-L GND #PWR?
+L GND #PWR03
 U 1 1 56D626D2
 P 6250 3900
-F 0 "#PWR?" H 6250 3900 30  0001 C CNN
+F 0 "#PWR03" H 6250 3900 30  0001 C CNN
 F 1 "GND" H 6250 3830 30  0001 C CNN
 F 2 "" H 6250 3900 60  0000 C CNN
@@
 $EndComp
 $Comp
-L GND #PWR?
+L GND #PWR04
 U 1 1 56D626E1
 P 4750 3700
-F 0 "#PWR?" H 4750 3700 30  0001 C CNN
+F 0 "#PWR04" H 4750 3700 30  0001 C CNN
 F 1 "GND" H 4750 3630 30  0001 C CNN
 F 2 "" H 4750 3700 60  0000 C CNN
