File: kicad/testadapter/testadapter.sch (KiCad schematic (older format))
At the start: 5 parts

Commit message: Created adapter PCB for testing sensorpods
Parts:
- added Q1, Q2, Q3: IRFML8244TRPBF, SOT-23, symbol IRFML8244TRPBF
- added R1, R2, R3: GENERIC_RESISTOR, 0805, symbol GENERIC_RESISTOR
- P1: renamed from P?; footprint ~ -> Header_5x2
- P2, P3, P4, P5: renamed from P?; footprint ~ -> Header_4x2
Connections:
- net labels added: +3.3V, +5V, Clock, GND, Load, NeoPixels
- wire segments 0 -> 81
- no-connect marks 0 -> 4
Other:
- moved on the sheet: P2, P3, P4, P5
